File: eagle_files/learning_zumo.sch (EAGLE design)
At the start: 27 parts, among them U1 3v3_Reg, U2 5V_Reg

Commit message: reflects most recent pcb changes
Connections:
- net IR_LED: now also U$1.36.D18
Changed lines of the file:
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@@
 <label x="68.58" y="71.12" size="1.778" layer="95"/>
+</segment>
+<segment>
+<pinref part="U$1" gate="G$1" pin="36.D18"/>
+<wire x1="154.94" y1="43.18" x2="165.1" y2="43.18" width="0.1524" layer="91"/>
+<label x="160.02" y="43.18" size="1.778" layer="95"/>
 </segment>
 </net>
