File: eagle_files/scratch/learning_zumo.brd (EAGLE design)
At the start: 66 x 66.4 mm, 68 parts, among them M1 DC_MOTOR, M2 DC_MOTOR, Y1 CRYSTAL-24MHZ, Y2 CRYSTAL-32KHZ

Commit message: latest WORKING version of board and schematic
Parts:
- removed C15: (no value), Swarm:E2,5-6
- removed U$2: GP2Y_DIST_SENSE_BREAKOUT, learning_particle:1X03
- added DIST_0, DIST_1: GP2Y_DIST_SENSE_BREAKOUT, learning_particle:1X03
- L6: device learning_particle:L0402_US -> learning_particle:R0805
- moved C32 7.07 mm to (12.0, 45.0), turned to 0 degrees
- moved C33 5.28 mm to (54.0, 45.0), turned to 0 degrees
- moved M1 5.16 mm to (18.4, 45.0)
- moved M2 5.16 mm to (47.6, 45.0)
- moved C23 1.98 mm to (30.2, 48.7)
- moved L6 1.33 mm to (32.2, 47.6)
- moved C19 0.30 mm to (28.4, 40.6)
Connections:
- removed net N$9: U$1.43
- new net DIST_1: DIST_1.SIG, U$1.43
- net 3V3: now also DIST_0.VCC, DIST_1.VCC, FB.P$1; no longer PW_SW.1.COMM, U$2.VCC
- net DCDC_SW: now also L6.1; no longer L6.P$1
- net DIST0: now also DIST_0.SIG; no longer U$2.SIG
- net GND: now also DIST_0.GND, DIST_1.GND; no longer C15.-, U$2.GND
- net N$4: now also 5V_REG.INPUT; no longer FB.P$1
- net VBAT: now also PW_SW.1.COMM; no longer 5V_REG.INPUT, C15.+
- net VDDR: now also L6.2; no longer L6.P$2
Routing:
- net DIST_1: track 0.00 -> 52.5 mm, vias 0 -> 2
- net DIST0: track 15.4 -> 53.0 mm, vias 0 -> 2
- net N$4: track 20.2 -> 54.1 mm, vias 0 -> 1
- net VBAT: track 72.3 -> 52.2 mm, vias 7 -> 3
- net 3V3: track 71.8 -> 60.5 mm
- net GND: track 45.2 -> 55.8 mm, vias 7 -> 9
- net N$26: track 33.2 -> 25.6 mm
- net N$25: track 31.1 -> 24.2 mm
- net N$27: track 32.4 -> 27.4 mm
- net N$24: track 30.7 -> 27.6 mm
- net DCDC_SW: track 1.42 -> 2.27 mm
- net VDDS: track 37.9 -> 37.2 mm
- net VDDR: track 20.3 -> 20.9 mm
Other:
- board text added: "v2.1 August 2020"
- board text removed: "v2.0 July 2020"
